Commit message: feat(robotiq_description): keep PickNik's sim_isaac arguments as deprecated aliases
sim_isaac, isaac_joint_commands and isaac_joint_states shipped in 1.1.0 and
are upstream's names. Without an alias `sim_isaac:=true` was still accepted
after the rename and silently started the real driver on /dev/ttyUSB0. The
launch file and both gripper macros now map the three onto sim_topic_based /
sim_joint_commands_topic / sim_joint_states_topic and warn (launch logger,
xacro.warning), sim_isaac restoring its old /isaac_joint_* topic defaults so
a 1.1.0 command line or URDF drives the same simulator. An explicit new-style
argument wins over both. Removed in the next major release.

Co-Authored-By: Claude Fable 5.1 <noreply@anthropic.com>

File: grippers/robotiq_description/urdf/robotiq_2f_140_macro.urdf.xacro (robot description, xacro)
@@ -10,4 +10,7 @@
         sim_joint_commands_topic:=/sim/joint_commands
         sim_joint_states_topic:=/sim/joint_states
+        sim_isaac:=false
+        isaac_joint_commands:=''
+        isaac_joint_states:=''
         use_fake_hardware:=false
         mock_sensor_commands:=false
@@ -20,4 +23,13 @@
         gripper_max_force:=125.0
         gripper_closed_position:=0.695">
+        <!-- PickNik's names for the topic-based path, released in 1.1.0 and
+             deprecated since 1.2.0. sim_isaac keeps its old /isaac_joint_* topic
+             defaults; an explicit new-style argument wins over both. -->
+        <xacro:if value="${sim_isaac or isaac_joint_commands != '' or isaac_joint_states != ''}">
+            ${xacro.warning('sim_isaac, isaac_joint_commands and isaac_joint_states are deprecated since 1.2.0 and removed in the next major release; use sim_topic_based, sim_joint_commands_topic and sim_joint_states_topic')}
+        </xacro:if>
+        <xacro:property name="topic_based" value="${sim_topic_based or sim_isaac}"/>
+        <xacro:property name="commands_topic" value="${isaac_joint_commands or ('/isaac_joint_commands' if sim_isaac else sim_joint_commands_topic)}"/>
+        <xacro:property name="states_topic" value="${isaac_joint_states or ('/isaac_joint_states' if sim_isaac else sim_joint_states_topic)}"/>
         <!-- ros2 control include -->
         <xacro:include filename="$(find robotiq_description)/urdf/2f_140.ros2_control.xacro" />
@@ -27,7 +39,7 @@
                 name="${name}" prefix="${prefix}"
                 sim_gazebo="${sim_gazebo}"
-                sim_topic_based="${sim_topic_based}"
-                sim_joint_commands_topic="${sim_joint_commands_topic}"
-                sim_joint_states_topic="${sim_joint_states_topic}"
+                sim_topic_based="${topic_based}"
+                sim_joint_commands_topic="${commands_topic}"
+                sim_joint_states_topic="${states_topic}"
                 use_fake_hardware="${use_fake_hardware}"
                 mock_sensor_commands="${mock_sensor_commands}"

File: grippers/robotiq_description/urdf/robotiq_2f_85_macro.urdf.xacro (robot description, xacro)
@@ -10,4 +10,7 @@
         sim_joint_commands_topic:=/sim/joint_commands
         sim_joint_states_topic:=/sim/joint_states
+        sim_isaac:=false
+        isaac_joint_commands:=''
+        isaac_joint_states:=''
         use_fake_hardware:=false
         mock_sensor_commands:=false
@@ -20,4 +23,13 @@
         gripper_max_force:=235.0
         gripper_closed_position:=0.7929">
+        <!-- PickNik's names for the topic-based path, released in 1.1.0 and
+             deprecated since 1.2.0. sim_isaac keeps its old /isaac_joint_* topic
+             defaults; an explicit new-style argument wins over both. -->
+        <xacro:if value="${sim_isaac or isaac_joint_commands != '' or isaac_joint_states != ''}">
+            ${xacro.warning('sim_isaac, isaac_joint_commands and isaac_joint_states are deprecated since 1.2.0 and removed in the next major release; use sim_topic_based, sim_joint_commands_topic and sim_joint_states_topic')}
+        </xacro:if>
+        <xacro:property name="topic_based" value="${sim_topic_based or sim_isaac}"/>
+        <xacro:property name="commands_topic" value="${isaac_joint_commands or ('/isaac_joint_commands' if sim_isaac else sim_joint_commands_topic)}"/>
+        <xacro:property name="states_topic" value="${isaac_joint_states or ('/isaac_joint_states' if sim_isaac else sim_joint_states_topic)}"/>
         <!-- ros2 control include -->
         <xacro:include filename="$(find robotiq_description)/urdf/2f_85.ros2_control.xacro" />
@@ -27,7 +39,7 @@
                 name="${name}" prefix="${prefix}"
                 sim_gazebo="${sim_gazebo}"
-                sim_topic_based="${sim_topic_based}"
-                sim_joint_commands_topic="${sim_joint_commands_topic}"
-                sim_joint_states_topic="${sim_joint_states_topic}"
+                sim_topic_based="${topic_based}"
+                sim_joint_commands_topic="${commands_topic}"
+                sim_joint_states_topic="${states_topic}"
                 use_fake_hardware="${use_fake_hardware}"
                 mock_sensor_commands="${mock_sensor_commands}"

File: grippers/robotiq_description/urdf/robotiq_2f_gripper.urdf.xacro (robot description, xacro)
@@ -12,4 +12,8 @@
     <xacro:arg name="sim_joint_commands_topic" default="/sim/joint_commands" />
     <xacro:arg name="sim_joint_states_topic" default="/sim/joint_states" />
+    <!-- Deprecated since 1.2.0, PickNik's names; the macro warns and maps them. -->
+    <xacro:arg name="sim_isaac" default="false" />
+    <xacro:arg name="isaac_joint_commands" default="" />
+    <xacro:arg name="isaac_joint_states" default="" />
     <!-- Import macros -->
     <xacro:include filename="$(find robotiq_description)/urdf/robotiq_$(arg gripper_model)_macro.urdf.xacro" />
@@ -17,5 +21,6 @@
     <xacro:robotiq_gripper name="RobotiqGripperHardwareInterface" prefix="" parent="world" use_fake_hardware="$(arg use_fake_hardware)" com_port="$(arg com_port)" baudrate="$(arg baudrate)"
         sim_topic_based="$(arg sim_topic_based)"
-        sim_joint_commands_topic="$(arg sim_joint_commands_topic)" sim_joint_states_topic="$(arg sim_joint_states_topic)">
+        sim_joint_commands_topic="$(arg sim_joint_commands_topic)" sim_joint_states_topic="$(arg sim_joint_states_topic)"
+        sim_isaac="$(arg sim_isaac)" isaac_joint_commands="$(arg isaac_joint_commands)" isaac_joint_states="$(arg isaac_joint_states)">
         <origin xyz="0 0 0" rpy="0 0 0" />
     </xacro:robotiq_gripper>
