Commit message: refactor(robotiq_description): drop the 2F prefix from the shared ros2_control block
- rename 2f_common.ros2_control.xacro to common.ros2_control.xacro, its macros to robotiq_hardware / robotiq_sim_mimic_joint

Co-Authored-By: Claude Opus 5.5 <noreply@anthropic.com>

File: grippers/robotiq_description/urdf/2f_140.ros2_control.xacro (robot description, xacro)
@@ -1,5 +1,5 @@
 <?xml version="1.0"?>
 <robot xmlns:xacro="http://www.ros.org/wiki/xacro">
-    <xacro:include filename="$(find robotiq_description)/urdf/2f_common.ros2_control.xacro" />
+    <xacro:include filename="$(find robotiq_description)/urdf/common.ros2_control.xacro" />
     <xacro:macro name="robotiq_gripper_ros2_control" params="
         name
@@ -20,5 +20,5 @@
         <ros2_control name="${name}" type="system">
             <!-- Plugins -->
-            <xacro:robotiq_2f_hardware
+            <xacro:robotiq_hardware
                 sim_gazebo="${sim_gazebo}"
                 sim_topic_based="${sim_topic_based}"
@@ -56,9 +56,9 @@
             <!-- When simulating we need to include the rest of the gripper joints -->
             <xacro:if value="${sim_topic_based or sim_gazebo}">
-                <xacro:robotiq_2f_sim_mimic_joint name="${prefix}left_inner_knuckle_joint" sim_gazebo="${sim_gazebo}"/>
-                <xacro:robotiq_2f_sim_mimic_joint name="${prefix}left_inner_finger_joint" sim_gazebo="${sim_gazebo}"/>
-                <xacro:robotiq_2f_sim_mimic_joint name="${prefix}right_outer_knuckle_joint" sim_gazebo="${sim_gazebo}"/>
-                <xacro:robotiq_2f_sim_mimic_joint name="${prefix}right_inner_knuckle_joint" sim_gazebo="${sim_gazebo}"/>
-                <xacro:robotiq_2f_sim_mimic_joint name="${prefix}right_inner_finger_joint" sim_gazebo="${sim_gazebo}"/>
+                <xacro:robotiq_sim_mimic_joint name="${prefix}left_inner_knuckle_joint" sim_gazebo="${sim_gazebo}"/>
+                <xacro:robotiq_sim_mimic_joint name="${prefix}left_inner_finger_joint" sim_gazebo="${sim_gazebo}"/>
+                <xacro:robotiq_sim_mimic_joint name="${prefix}right_outer_knuckle_joint" sim_gazebo="${sim_gazebo}"/>
+                <xacro:robotiq_sim_mimic_joint name="${prefix}right_inner_knuckle_joint" sim_gazebo="${sim_gazebo}"/>
+                <xacro:robotiq_sim_mimic_joint name="${prefix}right_inner_finger_joint" sim_gazebo="${sim_gazebo}"/>
             </xacro:if>
             <!-- Only add this with fake hardware mode -->

File: grippers/robotiq_description/urdf/2f_85.ros2_control.xacro (robot description, xacro)
@@ -1,5 +1,5 @@
 <?xml version="1.0"?>
 <robot xmlns:xacro="http://www.ros.org/wiki/xacro">
-    <xacro:include filename="$(find robotiq_description)/urdf/2f_common.ros2_control.xacro" />
+    <xacro:include filename="$(find robotiq_description)/urdf/common.ros2_control.xacro" />
     <xacro:macro name="robotiq_gripper_ros2_control" params="
         name
@@ -20,5 +20,5 @@
         <ros2_control name="${name}" type="system">
             <!-- Plugins -->
-            <xacro:robotiq_2f_hardware
+            <xacro:robotiq_hardware
                 sim_gazebo="${sim_gazebo}"
                 sim_topic_based="${sim_topic_based}"
@@ -63,9 +63,9 @@
             <!-- When simulating we need to include the rest of the gripper joints -->
             <xacro:if value="${sim_topic_based or sim_gazebo}">
-                <xacro:robotiq_2f_sim_mimic_joint name="${prefix}robotiq_85_right_knuckle_joint" sim_gazebo="${sim_gazebo}"/>
-                <xacro:robotiq_2f_sim_mimic_joint name="${prefix}robotiq_85_left_inner_knuckle_joint" sim_gazebo="${sim_gazebo}"/>
-                <xacro:robotiq_2f_sim_mimic_joint name="${prefix}robotiq_85_right_inner_knuckle_joint" sim_gazebo="${sim_gazebo}"/>
-                <xacro:robotiq_2f_sim_mimic_joint name="${prefix}robotiq_85_left_finger_tip_joint" sim_gazebo="${sim_gazebo}"/>
-                <xacro:robotiq_2f_sim_mimic_joint name="${prefix}robotiq_85_right_finger_tip_joint" sim_gazebo="${sim_gazebo}"/>
+                <xacro:robotiq_sim_mimic_joint name="${prefix}robotiq_85_right_knuckle_joint" sim_gazebo="${sim_gazebo}"/>
+                <xacro:robotiq_sim_mimic_joint name="${prefix}robotiq_85_left_inner_knuckle_joint" sim_gazebo="${sim_gazebo}"/>
+                <xacro:robotiq_sim_mimic_joint name="${prefix}robotiq_85_right_inner_knuckle_joint" sim_gazebo="${sim_gazebo}"/>
+                <xacro:robotiq_sim_mimic_joint name="${prefix}robotiq_85_left_finger_tip_joint" sim_gazebo="${sim_gazebo}"/>
+                <xacro:robotiq_sim_mimic_joint name="${prefix}robotiq_85_right_finger_tip_joint" sim_gazebo="${sim_gazebo}"/>
             </xacro:if>
             <!-- Only add this with fake hardware mode -->

File: grippers/robotiq_description/urdf/common.ros2_control.xacro (robot description, xacro)
@@ -1,8 +1,7 @@
 <?xml version="1.0"?>
 <robot xmlns:xacro="http://www.ros.org/wiki/xacro">
-    <!-- One <hardware> block shared by every 2F model. The joint names and
-         the per-model defaults stay in 2f_85.ros2_control.xacro /
-         2f_140.ros2_control.xacro. -->
-    <xacro:macro name="robotiq_2f_hardware" params="
+    <!-- One <hardware> block shared by every model. The joint names and the
+         per-model defaults stay in each <model>.ros2_control.xacro. -->
+    <xacro:macro name="robotiq_hardware" params="
         sim_gazebo
         sim_topic_based
@@ -50,5 +49,5 @@
          but never commanded. Gazebo derives mimic joints itself, so it gets no
          state interfaces either. -->
-    <xacro:macro name="robotiq_2f_sim_mimic_joint" params="name sim_gazebo">
+    <xacro:macro name="robotiq_sim_mimic_joint" params="name sim_gazebo">
         <joint name="${name}">
             <xacro:unless value="${sim_gazebo}">
