Commit message: feat(robotiq_description): adapt the Hand-E description to this repo
- move the meshes to meshes/*/hand_e, after gripper_model; the convex hull nothing references stays out
- robotiq_hand_e_macro.urdf.xacro on the 2F macros' parameters; finger collision from the finger meshes instead of PickNik's unit boxes
- hand_e.ros2_control.xacro on the shared hardware block
- gripper_model:=hand_e drives hande_finger_distance; the launch loads robotiq_gripper.urdf.xacro by default
- run the URDF and launch tests on the Hand-E

Co-Authored-By: Claude Opus 5.5 <noreply@anthropic.com>

File: grippers/robotiq_description/urdf/hand_e.ros2_control.xacro (robot description, xacro)
@@ -1,69 +1,65 @@
-<?xml version="1.0" encoding="UTF-8"?>
-<robot xmlns:xacro="http://wiki.ros.org/xacro">
-  <xacro:macro name="robotiq_hande_ros2_control" params="
-               name
-               prefix
-               sim_gazebo:=false
-               sim_isaac:=false
-               isaac_joint_commands:=/isaac_joint_commands
-               isaac_joint_states:=/isaac_joint_states
-               use_mock_hardware:=^|true
-               mock_sensor_commands:=^|true
-               com_port:=/dev/ttyUSB0">
-    <ros2_control name="${name}" type="system">
-      <hardware>
-        <xacro:if value="${sim_isaac}">
-          <plugin>topic_based_ros2_control/TopicBasedSystem</plugin>
-          <param name="joint_commands_topic">${isaac_joint_commands}</param>
-          <param name="joint_states_topic">${isaac_joint_states}</param>
-        </xacro:if>
-        <xacro:if value="${sim_gazebo}">
-          <plugin>gz_ros2_control/GzSystem</plugin>
-        </xacro:if>
-        <xacro:if value="${use_mock_hardware}">
-          <plugin>mock_components/GenericSystem</plugin>
-          <param name="mock_sensor_commands">${mock_sensor_commands}</param>
-        </xacro:if>
-        <xacro:unless value="${use_mock_hardware}">
-          <plugin>robotiq_driver/RobotiqGripperHardwareInterface</plugin>
-          <!-- default data from docs - https://blog.robotiq.com/hubfs/support-files/Hand-E_Adaptive_Gripper_ProductSheet_EN_2024-05_WEB.pdf -->
-          <param name="COM_port">${com_port}</param>
-          <param name="gripper_protocol_min_pos_value">0</param>
-          <param name="gripper_protocol_max_pos_value">255</param>
-          <param name="gripper_closed_position">0.05</param> <!-- usually the gripper's max stroke -->
-          <param name="max_speed">0.150</param>   <!-- m/s -->
-          <param name="speed_multiplier">1.0</param>
-          <param name="max_force">185.0</param>   <!-- N -->
-          <param name="force_multiplier">0.5</param>
-        </xacro:unless>
-      </hardware>
-      <joint name="${prefix}hande_finger_distance">
-        <command_interface name="position">
-          <param name="min">0.0</param>
-          <param name="max">0.050</param>
-        </command_interface>
-        <state_interface name="position">
-          <param name="initial_value">0.0</param>
-        </state_interface>
-        <state_interface name="velocity">
-          <param name="initial_value">0.0</param>
-        </state_interface>
-        <command_interface name="set_gripper_max_velocity">
-          <param name="min">0.020</param>
-          <param name="max">0.150</param>
-        </command_interface>
-        <command_interface name="set_gripper_max_effort">
-          <param name="min">20</param>
-          <param name="max">185</param>
-        </command_interface>
-      </joint>
-      <!-- Only add this with real and mock hardware mode -->
-      <xacro:unless value="${sim_gazebo or sim_isaac}">
-        <gpio name="reactivate_gripper">
-          <command_interface name="reactivate_gripper_cmd" />
-          <command_interface name="reactivate_gripper_response" />
-        </gpio>
-      </xacro:unless>
-    </ros2_control>
-  </xacro:macro>
+<?xml version="1.0"?>
+<robot xmlns:xacro="http://www.ros.org/wiki/xacro">
+    <xacro:include filename="$(find robotiq_description)/urdf/common.ros2_control.xacro" />
+    <xacro:macro name="robotiq_gripper_ros2_control" params="
+        name
+        prefix
+        sim_gazebo:=false
+        sim_topic_based:=false
+        sim_joint_commands_topic:=/sim/joint_commands
+        sim_joint_states_topic:=/sim/joint_states
+        use_fake_hardware:=false
+        mock_sensor_commands:=false
+        com_port:=/dev/ttyUSB0
+        baudrate:=115200
+        gripper_speed_multiplier:=1.0
+        gripper_force_multiplier:=0.5
+        gripper_max_speed:=0.150
+        gripper_max_force:=185.0
+        gripper_closed_position:=0.050">
+        <ros2_control name="${name}" type="system">
+            <xacro:robotiq_hardware
+                sim_gazebo="${sim_gazebo}"
+                sim_topic_based="${sim_topic_based}"
+                sim_joint_commands_topic="${sim_joint_commands_topic}"
+                sim_joint_states_topic="${sim_joint_states_topic}"
+                use_fake_hardware="${use_fake_hardware}"
+                mock_sensor_commands="${mock_sensor_commands}"
+                com_port="${com_port}"
+                baudrate="${baudrate}"
+                gripper_speed_multiplier="${gripper_speed_multiplier}"
+                gripper_force_multiplier="${gripper_force_multiplier}"
+                gripper_max_speed="${gripper_max_speed}"
+                gripper_max_force="${gripper_max_force}"
+                gripper_closed_position="${gripper_closed_position}"/>
+            <joint name="${prefix}hande_finger_distance">
+                <command_interface name="position" />
+                <!-- Mock-only; see the same block in 2f_85.ros2_control.xacro. -->
+                <xacro:if value="${use_fake_hardware}">
+                    <command_interface name="set_gripper_max_velocity"/>
+                    <command_interface name="set_gripper_max_effort"/>
+                </xacro:if>
+                <state_interface name="position">
+                    <param name="initial_value">0.0</param>
+                </state_interface>
+                <state_interface name="velocity"/>
+                <xacro:unless value="${use_fake_hardware or sim_gazebo or sim_topic_based}">
+                    <state_interface name="motor_current"/>
+                    <state_interface name="object_status"/>
+                    <state_interface name="gripper_fault"/>
+                    <state_interface name="gripper_fault_severity"/>
+                </xacro:unless>
+            </joint>
+            <xacro:if value="${sim_topic_based or sim_gazebo}">
+                <xacro:robotiq_sim_mimic_joint name="${prefix}hande_left_finger_joint" sim_gazebo="${sim_gazebo}"/>
+                <xacro:robotiq_sim_mimic_joint name="${prefix}hande_right_finger_joint" sim_gazebo="${sim_gazebo}"/>
+            </xacro:if>
+            <xacro:unless value="${sim_gazebo or sim_topic_based}">
+                <gpio name="reactivate_gripper">
+                    <command_interface name="reactivate_gripper_cmd" />
+                    <command_interface name="reactivate_gripper_response" />
+                </gpio>
+            </xacro:unless>
+        </ros2_control>
+    </xacro:macro>
 </robot>

File: grippers/robotiq_description/urdf/robotiq_gripper.urdf.xacro (robot description, xacro)
@@ -2,5 +2,5 @@
 <robot xmlns:xacro="http://wiki.ros.org/xacro" name="robotiq_gripper">
     <!-- parameters -->
-    <!-- gripper_model selects the macro (2f_85 / 2f_140). xacro args are
+    <!-- gripper_model selects the macro (2f_85 / 2f_140 / hand_e). xacro args are
          first-declaration-wins, so each wrapper must declare it BEFORE
          including this file, or the default below silently wins. -->

File: grippers/robotiq_description/urdf/robotiq_hand_e_gripper.urdf.xacro (robot description, xacro)
@@ -1,20 +1,5 @@
-<?xml version="1.0" encoding="UTF-8"?>
-<robot xmlns:xacro="http://wiki.ros.org/xacro" name="schunk_gripper">
-  <!-- Use this if parameters are set from the launch file, otherwise delete -->
-  <xacro:arg name="prefix" default="" />
-  <xacro:arg name="use_mock_hardware" default="false" />
-  <xacro:arg name="mock_sensor_commands" default="false" />
-  <xacro:include filename="$(find robotiq_description)/urdf/robotiq_hand_e_macro.urdf.xacro"/>
-  <xacro:include filename="$(find robotiq_description)/urdf/hand_e.ros2_control.xacro"/>
-  <!-- create link fixed to the "world" -->
-  <link name="base_link" />
-  <!-- Load robot's macro with parameters -->
-  <!-- set prefix if multiple robots are used -->
-  <xacro:robotiq_hande prefix="$(arg prefix)" parent="base_link" >
-    <origin xyz="0 0 0" rpy="0 0 0" />          <!-- position robot in the world -->
-  </xacro:robotiq_hande>
-  <xacro:robotiq_hande_ros2_control
-    name="robotiq_hande"
-    prefix="$(arg prefix)"
-    use_mock_hardware="$(arg use_mock_hardware)" />
+<?xml version="1.0"?>
+<robot xmlns:xacro="http://wiki.ros.org/xacro" name="robotiq_gripper">
+    <xacro:arg name="gripper_model" default="hand_e" />
+    <xacro:include filename="$(find robotiq_description)/urdf/robotiq_gripper.urdf.xacro" />
 </robot>
