Commit message: feat(robotiq_description): adapt the Hand-E description to this repo
- move the meshes to meshes/*/hand_e, after gripper_model; the convex hull nothing references stays out
- robotiq_hand_e_macro.urdf.xacro on the 2F macros' parameters; finger collision from the finger meshes instead of PickNik's unit boxes
- hand_e.ros2_control.xacro on the shared hardware block
- gripper_model:=hand_e drives hande_finger_distance; the launch loads robotiq_gripper.urdf.xacro by default
- run the URDF and launch tests on the Hand-E

Co-Authored-By: Claude Opus 5.5 <noreply@anthropic.com>

File: grippers/robotiq_description/urdf/robotiq_hand_e_macro.urdf.xacro (robot description, xacro)
@@ -1,143 +1,143 @@
 <?xml version="1.0"?>
-<robot xmlns:xacro="http://www.ros.org/wiki/xacro" name="gripper_finger">
-    <!-- Colour definations-->
-    <material name="gray">
-      <color rgba="0.7 0.7 0.7 1.0"/>
-    </material>
-    <material name="dark">
-      <color rgba=".1 0.1 0.1 1.0"/>
-    </material>
-    <!-- Gripper macro hand-e -->
-    <xacro:macro name="robotiq_hande" params="
-                 prefix parent *origin
-                 left_finger_visual:=default left_finger_collision:=default
-                 left_finger_scale:=default left_finger_collision_scale:=default
-                 right_finger_visual:=default right_finger_collision:=default
-                 right_finger_scale:=default right_finger_collision_scale:=default
-                 tcp_z_offset:=0.1325
-                 ">
-      <xacro:property name="file_path" value="file://$(find robotiq_description)" />
-      <xacro:property name="gripper_maximal_stroke" value="0.050" />
-      <!-- resolve complex default values -->
-      <xacro:if value="${left_finger_visual == 'default'}">
-        <xacro:property name="left_finger_visual" value="${file_path}/meshes/visual/hande/left_finger.dae" />
-      </xacro:if>
-      <xacro:if value="${left_finger_collision == 'default'}">
-        <xacro:property name="left_finger_collision" value="${file_path}/meshes/collision/hande/left_finger.stl" />
-      </xacro:if>
-      <xacro:if value="${left_finger_scale == 'default'}">
-        <xacro:property name="left_finger_scale" value="1.0 1.0 1.0" />
-      </xacro:if>
-      <xacro:if value="${left_finger_collision_scale == 'default'}">
-        <xacro:property name="left_finger_collision_scale" value="1.0 1.0 1.0" />
-      </xacro:if>
-      <xacro:if value="${right_finger_visual == 'default'}">
-        <xacro:property name="right_finger_visual" value="${file_path}/meshes/visual/hande/right_finger.dae" />
-      </xacro:if>
-      <xacro:if value="${right_finger_collision == 'default'}">
-        <xacro:property name="right_finger_collision" value="${file_path}/meshes/collision/hande/right_finger.stl" />
-      </xacro:if>
-      <xacro:if value="${right_finger_collision_scale == 'default'}">
-        <xacro:property name="right_finger_scale" value="1.0 1.0 1.0" />
-      </xacro:if>
-      <xacro:if value="${right_finger_collision_scale == 'default'}">
-        <xacro:property name="right_finger_collision_scale" value="1.0 1.0 1.0" />
-      </xacro:if>
-      <link name="${prefix}hand_e_base_link">
-          <inertial>
-            <origin rpy="0 0 0" xyz="0 0 0.04607"/>
-            <mass value="0.86387"/>
-            <inertia ixx="1017560E-9" ixy="0" ixz="2235E-9" iyy="1028041E-9" iyz="0" izz="489810E-9"/>
-          </inertial>
-          <visual>
-              <origin rpy="0 0 0" xyz="0 0 0"/>
-              <geometry>
-                  <mesh filename="${file_path}/meshes/visual/hande/hand-e.dae" scale="1.0 1.0 1.0"/>
-              </geometry>
-              <material name="dark" />
-          </visual>
-          <collision>
-              <origin rpy="0 0 0" xyz="0 0 0"/>
-              <geometry>
-                  <mesh filename="${file_path}/meshes/collision/hande/hand-e.stl" scale="1.0 1.0 1.0"/>
-                  <!--<mesh filename="${file_path}/meshes/collision/hande/hand-e_convex_hull.stl" scale="1.0 1.0 1.0"/>-->
-              </geometry>
-          </collision>
-      </link>
-      <joint name="${prefix}robotiq_hande_base_joint" type="fixed">
-          <parent link="${parent}"/>
-          <child link="${prefix}hand_e_base_link"/>
-          <xacro:insert_block name="origin"/>
-      </joint>
-      <!-- Fingers -->
-      <link name="${prefix}hande_left_finger">
-          <visual>
-            <origin rpy="0 0 0" xyz="0 0 0"/>
-            <geometry>
-              <mesh filename="${left_finger_visual}" scale="${left_finger_scale}" />
-            </geometry>
-            <material name="gray">
-              <color rgba="0.7 0.7 0.7 1.0"/>
-            </material>
-          </visual>
-          <collision>
-            <origin rpy="0 0 0" xyz="${-0.010} ${-0.075/2} ${0.028/2}"/>
-            <geometry>
-<!--               <mesh filename="${left_finger_collision}" scale="1.0 1.0 1.0" /> -->
-              <box size="${left_finger_collision_scale}" />
-            </geometry>
-          </collision>
+<robot xmlns:xacro="http://wiki.ros.org/xacro" name="robotiq_gripper">
+    <xacro:macro name="robotiq_gripper" params="
+        name
+        prefix
+        parent
+        *origin
+        sim_gazebo:=false
+        sim_topic_based:=false
+        sim_joint_commands_topic:=/sim/joint_commands
+        sim_joint_states_topic:=/sim/joint_states
+        sim_isaac:=false
+        isaac_joint_commands:=''
+        isaac_joint_states:=''
+        use_fake_hardware:=false
+        mock_sensor_commands:=false
+        include_ros2_control:=true
+        com_port:=/dev/ttyUSB0
+        baudrate:=115200
+        gripper_speed_multiplier:=1.0
+        gripper_force_multiplier:=0.5
+        gripper_max_speed:=0.150
+        gripper_max_force:=185.0
+        gripper_closed_position:=0.050
+        tcp_z_offset:=0.1325">
+        <!-- PickNik's names for the topic-based path, released in 1.1.0 and
+             deprecated since 1.2.0. sim_isaac keeps its old /isaac_joint_* topic
+             defaults; an explicit new-style argument wins over both. -->
+        <xacro:if value="${sim_isaac or isaac_joint_commands != '' or isaac_joint_states != ''}">
+            ${xacro.warning('sim_isaac, isaac_joint_commands and isaac_joint_states are deprecated since 1.2.0 and removed in the next major release; use sim_topic_based, sim_joint_commands_topic and sim_joint_states_topic')}
+        </xacro:if>
+        <xacro:property name="topic_based" value="${sim_topic_based or sim_isaac}"/>
+        <xacro:property name="commands_topic" value="${isaac_joint_commands or ('/isaac_joint_commands' if sim_isaac else sim_joint_commands_topic)}"/>
+        <xacro:property name="states_topic" value="${isaac_joint_states or ('/isaac_joint_states' if sim_isaac else sim_joint_states_topic)}"/>
+        <xacro:property name="stroke" value="0.050"/>
+        <xacro:include filename="$(find robotiq_description)/urdf/hand_e.ros2_control.xacro" />
+        <xacro:if value="${include_ros2_control}">
+            <xacro:robotiq_gripper_ros2_control
+                name="${name}" prefix="${prefix}"
+                sim_gazebo="${sim_gazebo}"
+                sim_topic_based="${topic_based}"
+                sim_joint_commands_topic="${commands_topic}"
+                sim_joint_states_topic="${states_topic}"
+                use_fake_hardware="${use_fake_hardware}"
+                mock_sensor_commands="${mock_sensor_commands}"
+                com_port="${com_port}"
+                baudrate="${baudrate}"
+                gripper_speed_multiplier="${gripper_speed_multiplier}"
+                gripper_force_multiplier="${gripper_force_multiplier}"
+                gripper_max_speed="${gripper_max_speed}"
+                gripper_max_force="${gripper_max_force}"
+                gripper_closed_position="${gripper_closed_position}"/>
+        </xacro:if>
+        <link name="${prefix}hand_e_base_link">
+            <inertial>
+                <origin xyz="0 0 0.04607" rpy="0 0 0" />
+                <mass value="0.86387" />
+                <inertia ixx="1017560E-9" ixy="0" ixz="2235E-9" iyy="1028041E-9" iyz="0" izz="489810E-9" />
+            </inertial>
+            <visual>
+                <geometry>
+                    <mesh filename="package://robotiq_description/meshes/visual/hand_e/hand-e.dae" />
+                </geometry>
+                <material name="">
+                    <color rgba="0.1 0.1 0.1 1" />
+                </material>
+            </visual>
+            <collision>
+                <geometry>
+                    <mesh filename="package://robotiq_description/meshes/collision/hand_e/hand-e.stl" />
+                </geometry>
+            </collision>
+        </link>
+        <joint name="${prefix}robotiq_hande_base_joint" type="fixed">
+            <parent link="${parent}" />
+            <child link="${prefix}hand_e_base_link" />
+            <xacro:insert_block name="origin" />
+        </joint>
+        <link name="${prefix}hande_left_finger">
+            <visual>
+                <geometry>
+                    <mesh filename="package://robotiq_description/meshes/visual/hand_e/left_finger.dae" />
+                </geometry>
+                <material name="">
+                    <color rgba="0.7 0.7 0.7 1" />
+                </material>
+            </visual>
+            <collision>
+                <geometry>
+                    <mesh filename="package://robotiq_description/meshes/collision/hand_e/left_finger.stl" />
+                </geometry>
+            </collision>
         </link>
         <link name="${prefix}hande_right_finger">
-          <visual>
-            <origin rpy="0 0 0" xyz="0 0 0"/>
-            <geometry>
-              <mesh filename="${right_finger_visual}" scale="${right_finger_scale}" />
-            </geometry>
-            <material name="gray">
-              <color rgba="0.7 0.7 0.7 1.0"/>
-            </material>
-          </visual>
-          <collision>
-            <origin rpy="0 0 0" xyz="${0.010} ${-0.075/2} ${0.028/2}"/>
-            <geometry>
-              <box size="${right_finger_collision_scale}" />
-<!--               <mesh filename="${right_finger_collision}" scale="1.0 1.0 1.0" /> -->
-            </geometry>
-          </collision>
-      </link>
-      <!-- virtual joint to model values coming from the gripper to the geometry - gripper uses
-      distance between fingers as command and state values -->
-      <link name="${prefix}hande_finger_distance_link" />
-      <joint name="${prefix}hande_finger_distance" type="prismatic">
-        <axis xyz="1 0 0"/>
-        <parent link="${prefix}hand_e_base_link"/>
-        <child link="${prefix}hande_finger_distance_link"/>
-        <origin rpy="0 0 0" xyz="0 0 0.099"/>
-        <axis xyz="1 0 0"/>
-        <limit effort="180" lower="0.0" upper="${gripper_maximal_stroke}" velocity="0.15"/>
-      </joint>
-      <joint name="${prefix}hande_left_finger_joint" type="prismatic">
-        <origin rpy="0 0 0" xyz="0 0 0.099"/>
-        <parent link="${prefix}hand_e_base_link"/>
-        <child link="${prefix}hande_left_finger"/>
-        <axis xyz="-1 0 0"/>
-        <limit effort="180" lower="0" upper="${gripper_maximal_stroke/2}" velocity="0.15"/>
-        <mimic joint="${prefix}hande_finger_distance" multiplier="-0.5" offset="${gripper_maximal_stroke/2}"/>
-      </joint>
-      <joint name="${prefix}hande_right_finger_joint" type="prismatic">
-        <origin rpy="0 0 0" xyz="0 0 0.099"/>
-        <parent link="${prefix}hand_e_base_link"/>
-        <child link="${prefix}hande_right_finger"/>
-        <axis xyz="1 0 0"/>
-        <limit effort="180" lower="0" upper="${gripper_maximal_stroke/2}" velocity="0.15"/>
-        <mimic joint="${prefix}hande_finger_distance" multiplier="-0.5" offset="${gripper_maximal_stroke/2}"/>
-      </joint>
-      <link name="${prefix}tcp_link"/>
-      <joint name="${prefix}tcp_link_joint" type="fixed">
-        <origin xyz="0 0 ${tcp_z_offset}" rpy="0 0 ${-pi/2}"/>
-        <parent link="${prefix}hand_e_base_link"/>
-        <child link="${prefix}tcp_link"/>
-      </joint>
+            <visual>
+                <geometry>
+                    <mesh filename="package://robotiq_description/meshes/visual/hand_e/right_finger.dae" />
+                </geometry>
+                <material name="">
+                    <color rgba="0.7 0.7 0.7 1" />
+                </material>
+            </visual>
+            <collision>
+                <geometry>
+                    <mesh filename="package://robotiq_description/meshes/collision/hand_e/right_finger.stl" />
+                </geometry>
+            </collision>
+        </link>
+        <!-- The driven joint has no geometry of its own: the gripper reports one
+             position for the pair, 0 open to the stroke closed, and each finger
+             travels half of it. -->
+        <link name="${prefix}hande_finger_distance_link" />
+        <joint name="${prefix}hande_finger_distance" type="prismatic">
+            <parent link="${prefix}hand_e_base_link" />
+            <child link="${prefix}hande_finger_distance_link" />
+            <axis xyz="1 0 0" />
+            <origin xyz="0 0 0.099" rpy="0 0 0" />
+            <limit lower="0.0" upper="${stroke}" velocity="0.15" effort="180" />
+        </joint>
+        <joint name="${prefix}hande_left_finger_joint" type="prismatic">
+            <parent link="${prefix}hand_e_base_link" />
+            <child link="${prefix}hande_left_finger" />
+            <axis xyz="-1 0 0" />
+            <origin xyz="0 0 0.099" rpy="0 0 0" />
+            <limit lower="0.0" upper="${stroke/2}" velocity="0.15" effort="180" />
+            <mimic joint="${prefix}hande_finger_distance" multiplier="-0.5" offset="${stroke/2}" />
+        </joint>
+        <joint name="${prefix}hande_right_finger_joint" type="prismatic">
+            <parent link="${prefix}hand_e_base_link" />
+            <child link="${prefix}hande_right_finger" />
+            <axis xyz="1 0 0" />
+            <origin xyz="0 0 0.099" rpy="0 0 0" />
+            <limit lower="0.0" upper="${stroke/2}" velocity="0.15" effort="180" />
+            <mimic joint="${prefix}hande_finger_distance" multiplier="-0.5" offset="${stroke/2}" />
+        </joint>
+        <link name="${prefix}tcp_link" />
+        <joint name="${prefix}tcp_link_joint" type="fixed">
+            <parent link="${prefix}hand_e_base_link" />
+            <child link="${prefix}tcp_link" />
+            <origin xyz="0 0 ${tcp_z_offset}" rpy="0 0 ${-pi/2}" />
+        </joint>
     </xacro:macro>
 </robot>

Commit message: feat(robotiq_description): adapt the Hand-E description to this repo
- move the meshes to meshes/*/hand_e, after gripper_model; the convex hull nothing references stays out
- robotiq_hand_e_macro.urdf.xacro on the 2F macros' parameters; finger collision from the finger meshes instead of PickNik's unit boxes
- hand_e.ros2_control.xacro on the shared hardware block with the hand_e profile, taking every argument from the macro instead of repeating its defaults
- hande_left_finger_joint is that finger's travel, 0 open to 0.025 m closed, like the 2F knuckle; the right finger mimics it, and PickNik's virtual hande_finger_distance goes
- gripper_model:=hand_e drives hande_left_finger_joint; the launch loads robotiq_gripper.urdf.xacro by default
- run the URDF and launch tests on the Hand-E

Co-Authored-By: Claude Opus 5.5 <noreply@anthropic.com>

File: grippers/robotiq_description/urdf/hand_e.ros2_control.xacro (robot description, xacro)
@@ -1,69 +1,67 @@
-<?xml version="1.0" encoding="UTF-8"?>
-<robot xmlns:xacro="http://wiki.ros.org/xacro">
-  <xacro:macro name="robotiq_hande_ros2_control" params="
-               name
-               prefix
-               sim_gazebo:=false
-               sim_isaac:=false
-               isaac_joint_commands:=/isaac_joint_commands
-               isaac_joint_states:=/isaac_joint_states
-               use_mock_hardware:=^|true
-               mock_sensor_commands:=^|true
-               com_port:=/dev/ttyUSB0">
-    <ros2_control name="${name}" type="system">
-      <hardware>
-        <xacro:if value="${sim_isaac}">
-          <plugin>topic_based_ros2_control/TopicBasedSystem</plugin>
-          <param name="joint_commands_topic">${isaac_joint_commands}</param>
-          <param name="joint_states_topic">${isaac_joint_states}</param>
-        </xacro:if>
-        <xacro:if value="${sim_gazebo}">
-          <plugin>gz_ros2_control/GzSystem</plugin>
-        </xacro:if>
-        <xacro:if value="${use_mock_hardware}">
-          <plugin>mock_components/GenericSystem</plugin>
-          <param name="mock_sensor_commands">${mock_sensor_commands}</param>
-        </xacro:if>
-        <xacro:unless value="${use_mock_hardware}">
-          <plugin>robotiq_driver/RobotiqGripperHardwareInterface</plugin>
-          <!-- default data from docs - https://blog.robotiq.com/hubfs/support-files/Hand-E_Adaptive_Gripper_ProductSheet_EN_2024-05_WEB.pdf -->
-          <param name="COM_port">${com_port}</param>
-          <param name="gripper_protocol_min_pos_value">0</param>
-          <param name="gripper_protocol_max_pos_value">255</param>
-          <param name="gripper_closed_position">0.05</param> <!-- usually the gripper's max stroke -->
-          <param name="max_speed">0.150</param>   <!-- m/s -->
-          <param name="speed_multiplier">1.0</param>
-          <param name="max_force">185.0</param>   <!-- N -->
-          <param name="force_multiplier">0.5</param>
-        </xacro:unless>
-      </hardware>
-      <joint name="${prefix}hande_finger_distance">
-        <command_interface name="position">
-          <param name="min">0.0</param>
-          <param name="max">0.050</param>
-        </command_interface>
-        <state_interface name="position">
-          <param name="initial_value">0.0</param>
-        </state_interface>
-        <state_interface name="velocity">
-          <param name="initial_value">0.0</param>
-        </state_interface>
-        <command_interface name="set_gripper_max_velocity">
-          <param name="min">0.020</param>
-          <param name="max">0.150</param>
-        </command_interface>
-        <command_interface name="set_gripper_max_effort">
-          <param name="min">20</param>
-          <param name="max">185</param>
-        </command_interface>
-      </joint>
-      <!-- Only add this with real and mock hardware mode -->
-      <xacro:unless value="${sim_gazebo or sim_isaac}">
-        <gpio name="reactivate_gripper">
-          <command_interface name="reactivate_gripper_cmd" />
-          <command_interface name="reactivate_gripper_response" />
-        </gpio>
-      </xacro:unless>
-    </ros2_control>
-  </xacro:macro>
+<?xml version="1.0"?>
+<robot xmlns:xacro="http://www.ros.org/wiki/xacro">
+    <xacro:include filename="$(find robotiq_description)/urdf/common.ros2_control.xacro" />
+    <!-- No defaults: the Hand-E's live in robotiq_hand_e_macro.urdf.xacro,
+         which passes every argument. -->
+    <xacro:macro name="robotiq_gripper_ros2_control" params="
+        name
+        prefix
+        sim_gazebo
+        sim_topic_based
+        sim_joint_commands_topic
+        sim_joint_states_topic
+        use_fake_hardware
+        mock_sensor_commands
+        com_port
+        baudrate
+        gripper_speed_multiplier
+        gripper_force_multiplier
+        gripper_max_speed
+        gripper_max_force
+        gripper_closed_position">
+        <ros2_control name="${name}" type="system">
+            <xacro:robotiq_hardware
+                sim_gazebo="${sim_gazebo}"
+                sim_topic_based="${sim_topic_based}"
+                sim_joint_commands_topic="${sim_joint_commands_topic}"
+                sim_joint_states_topic="${sim_joint_states_topic}"
+                use_fake_hardware="${use_fake_hardware}"
+                mock_sensor_commands="${mock_sensor_commands}"
+                com_port="${com_port}"
+                baudrate="${baudrate}"
+                gripper_speed_multiplier="${gripper_speed_multiplier}"
+                gripper_force_multiplier="${gripper_force_multiplier}"
+                gripper_max_speed="${gripper_max_speed}"
+                gripper_max_force="${gripper_max_force}"
+                gripper_closed_position="${gripper_closed_position}"
+                gripper_profile="hand_e"/>
+            <joint name="${prefix}hande_left_finger_joint">
+                <command_interface name="position" />
+                <!-- Mock-only; see the same block in 2f_85.ros2_control.xacro. -->
+                <xacro:if value="${use_fake_hardware}">
+                    <command_interface name="set_gripper_max_velocity"/>
+                    <command_interface name="set_gripper_max_effort"/>
+                </xacro:if>
+                <state_interface name="position">
+                    <param name="initial_value">0.0</param>
+                </state_interface>
+                <state_interface name="velocity"/>
+                <xacro:unless value="${use_fake_hardware or sim_gazebo or sim_topic_based}">
+                    <state_interface name="motor_current"/>
+                    <state_interface name="object_status"/>
+                    <state_interface name="gripper_fault"/>
+                    <state_interface name="gripper_fault_severity"/>
+                </xacro:unless>
+            </joint>
+            <xacro:if value="${sim_topic_based or sim_gazebo}">
+                <xacro:robotiq_sim_mimic_joint name="${prefix}hande_right_finger_joint" sim_gazebo="${sim_gazebo}"/>
+            </xacro:if>
+            <xacro:unless value="${sim_gazebo or sim_topic_based}">
+                <gpio name="reactivate_gripper">
+                    <command_interface name="reactivate_gripper_cmd" />
+                    <command_interface name="reactivate_gripper_response" />
+                </gpio>
+            </xacro:unless>
+        </ros2_control>
+    </xacro:macro>
 </robot>
